Commit message: update

File: src/rosmaster/description/rosmaster_core.xacro (robot description, xacro)
@@ -2,4 +2,19 @@
 <robot xmlns:xacro="http://www.ros.org/wiki/xacro">
 <xacro:include filename="inertial_macros.xacro"/>
+<material name="white">
+    <color rgba="1 1 1 1" />
+</material>
+<material name="orange">
+    <color rgba="1 0.3 0.1 1" />
+</material>
+<material name="blue">
+    <color rgba="0.2 0.2 1 1" />
+</material>
+<material name="black">
+    <color rgba="0 0 0 1" />
+</material>
+<material name="red">
+    <color rgba="1 0 0 1" />
+</material>
   <xacro:property name="wheel_radius" value="0.05"/>
   <xacro:property name="wheel_width" value="0.03"/>
@@ -15,17 +30,31 @@
 </link>
   <link name="base_link">
-    <inertial>
-      <mass value="5.0"/>
+  </link>
+  <joint name="chassis_joint" type="fixed">
+    <parent link="base_link"/>
+    <child link="chassis"/>
+    <origin xyz="0 0 0"/>
+  </joint>
+  <link name="chassis">
+    <visual>
       <origin xyz="0 0 0"/>
-      <inertia ixx="0.1" ixy="0.0" ixz="0.0"
-               iyy="0.1" iyz="0.0"
-               izz="0.1"/>
-    </inertial>
-    <visual>
       <geometry>
         <box size="0.4 0.3 0.1"/>
       </geometry>
+      <material name="white"/>
     </visual>
+    <collision>
+      <origin xyz="0 0 0"/>
+      <geometry>
+        <box size="0.4 0.3 0.1"/>
+      </geometry>
+    </collision>
+    <xacro:inertial_box mass="0.5" x="0" y="0" z="0">
+      <origin xyz="0 0 0" rpy="0 0 0"/>
+    </xacro:inertial_box>
   </link>
+  <gazebo reference="chassis">
+    <material>Gazebo/White</material>
+  </gazebo>
   <xacro:macro name="wheel" params="name x y">
     <link name="${name}_link">
@@ -35,12 +64,18 @@
         </geometry>
       </visual>
-      <inertial>
-        <mass value="0.5"/>
-        <origin xyz="0 0 0"/>
-        <inertia ixx="0.001" ixy="0.0" ixz="0.0"
-                 iyy="0.001" iyz="0.0"
-                 izz="0.001"/>
-      </inertial>
+      <collision>
+        <geometry>
+            <sphere radius="${wheel_radius}"/>
+        </geometry>
+      </collision>
+      <xacro:inertial_cylinder mass="0.5" length="${wheel_width}" radius="${wheel_radius}">
+          <origin xyz="0 0 0" rpy="0 0 0"/>
+      </xacro:inertial_cylinder>
     </link>
+    <gazebo reference="${name}_link">
+        <material>Gazebo/Blue</material>
+        <!-- <mu1 value="0.09"/>
+        <mu2 value="0.09"/> -->
+    </gazebo>
     <joint name="${name}_joint" type="continuous">
       <parent link="base_link"/>
